Commit message: calibrate right robot

File: calibrated_urdf/fr3_2/fr3.urdf (robot description, URDF)
Before this commit: robot fr3, 15 links, 14 joints
Joints:
- joint ball_joint: origin xyz=0.0005817897427710198 0.00017076431392279808 0.03181696256838364 rpy=0.0 0.0 0.0 -> xyz=0.0005730469232469997 0.00017246379341305678 0.03180233409997478 rpy=0.0 0.0 0.0
- joint fr3_finger_joint2: axis 0 -1 0 -> 0 1 0; origin xyz=0 0 0.0584 rpy=0 0 0 -> xyz=0 0 0.0584 rpy=0 0 3.141592653589793
- joint fr3_joint1: origin xyz=3.2503017915823636e-17 -1.0052584428671278e-17 0.333 rpy=9.835862032736894e-18 -1.568628146777241e-17 -9.300888715305458e-19 -> xyz=9.721333546283258e-17 -1.3633068073102069e-17 0.333 rpy=4.6680867266761446e-18 -4.3938331889645755e-17 6.921821648214007e-17
- joint fr3_joint2: origin xyz=-0.0002610630417672176 3.162243216911802e-05 6.491857691235396e-18 rpy=-1.5694399183345502 0.008109347349404753 1.0266954813848713e-06 -> xyz=-0.0002363665105483772 -2.3389096414359724e-05 9.345262340795115e-18 rpy=-1.569627770805241 0.008161719804770411 4.9969770548432846e-08
- joint fr3_joint3: origin xyz=0.002533495183565273 -0.31626197441515996 3.217901233781086e-05 rpy=1.5683189972748102 -0.0017477803894106437 0.00730424808627864 -> xyz=0.0025427422853042535 -0.31623620280060866 -2.3361244751523792e-05 rpy=1.5684060893837966 -0.0018168428316431508 0.007358035759455237
- joint fr3_joint4: origin xyz=0.08234090055495948 0.00040039919814801364 0.00028318793219997174 rpy=1.5676194275812498 0.001481487056437176 0.001736401255948335 -> xyz=0.08220728375338619 0.00039627327167539756 0.0002549472944480031 rpy=1.5677352970537977 0.001333182466844594 0.001801876443779632
- joint fr3_joint5: origin xyz=-0.08200856939548035 0.3847203771425275 -0.00040672740794162374 rpy=-1.5713567033269413 0.003565843461630894 -0.0012264927231521708 -> xyz=-0.08201728720917734 0.384725907132877 -0.0003963046312873375 rpy=-1.571397844929467 0.00351279731718852 -0.00108234741258956
- joint fr3_joint6: origin xyz=0.0006687445854766019 0.0003806617612789464 0.0007223020527509455 rpy=1.5661988055612805 3.25644008541223e-05 0.0035667292074115 -> xyz=0.0006845792932000495 0.00042484826435466595 0.0007267061230233097 rpy=1.5665350621383638 2.870446407541546e-05 0.003513514870217009
- joint fr3_joint7: origin xyz=0.08787630243262287 7.798120106991974e-06 -0.0003730253641811346 rpy=1.5708821891077023 3.5812492014648904e-07 -1.7024685193937513e-05 -> xyz=0.0878864823581289 -3.0718995970887753e-07 -0.0004191913496779998 rpy=1.5708893971925517 1.1434688315272071e-08 -1.379639019849125e-05

File: calibrated_urdf/fr3_2/step_0/model.urdf (robot description, URDF)
Before this commit: robot fr3, 15 links, 14 joints
Joints:
- joint ball_joint: origin xyz=0.000395598243266111 -7.962906613136055e-05 0.03180077705269587 rpy=0.0 0.0 0.0 -> xyz=7.773732033005863e-05 -4.214022515884392e-05 0.030128297908475325 rpy=0.0 0.0 0.0
- joint fr3_finger_joint2: axis 0 -1 0 -> 0 1 0; origin xyz=0 0 0.0584 rpy=0 0 0 -> xyz=0 0 0.0584 rpy=0 0 3.141592653589793

File: calibrated_urdf/fr3_2/step_1/model.urdf (robot description, URDF)
Before this commit: robot fr3, 15 links, 14 joints
Joints:
- joint ball_joint: origin xyz=0.0005601923688563379 0.00021286581312431914 0.03287437830668481 rpy=0.0 0.0 0.0 -> xyz=0.000527498949704872 0.0002222774642964122 0.032065948716657945 rpy=0.0 0.0 0.0
- joint fr3_finger_joint2: axis 0 -1 0 -> 0 1 0; origin xyz=0 0 0.0584 rpy=0 0 0 -> xyz=0 0 0.0584 rpy=0 0 3.141592653589793
- joint fr3_joint1: origin xyz=-3.4086023906813614e-17 1.0658678061771992e-17 0.33299999999999996 rpy=1.161626004634265e-17 4.578034837205634e-17 9.11091352262601e-17 -> xyz=5.252629276490508e-17 -2.3511750220720102e-17 0.3330000000000001 rpy=2.4201191891299292e-17 -7.457257524251103e-17 -1.613774001999991e-17
- joint fr3_joint2: origin xyz=-0.00034106902724989255 -0.0005581386978119321 -3.4650568716582776e-17 rpy=-1.5684849581257947 0.008815875083860706 0.0003725558057668295 -> xyz=-0.0002107446905017599 -0.000759777874866128 2.975080398450758e-17 rpy=-1.5677068306927149 0.009487967254328053 0.0005210031879156583
- joint fr3_joint3: origin xyz=0.002850207186231282 -0.3161988045741027 -0.00035400322520741335 rpy=1.5681072706125097 -0.00042682474338728664 0.006250789477593478 -> xyz=0.0029825638404374424 -0.3162013178792046 -0.00044247097064073937 rpy=1.5679478646629292 -0.00035077319796870466 0.0065915851472026265
- joint fr3_joint4: origin xyz=0.08240676263331533 -0.0003614305488879559 0.001200140980625334 rpy=1.5672686522171362 0.0016991644875519725 0.0017776812881444067 -> xyz=0.08244892849949022 -0.0005002381979472772 0.001398151797334963 rpy=1.5671474647743768 0.001816150665074235 0.001826355326540763
- joint fr3_joint5: origin xyz=-0.08249377125070924 0.38536015243170174 -0.0021933224572779626 rpy=-1.570909894346742 0.0030040694158974253 -0.0010836902771143757 -> xyz=-0.08265294356046765 0.3854690804571784 -0.0025440733135735807 rpy=-1.5709690714562161 0.00263915637202947 -0.0009303565118177015
- joint fr3_joint6: origin xyz=0.00041242759511092185 0.0009986960939698125 0.0017688756274369236 rpy=1.5688210427012124 -0.0005862974544913274 0.0030720501224883725 -> xyz=0.00033098157901070797 0.001452796925845996 0.0019031516426533401 rpy=1.5691520431572428 -0.0012064463144289854 0.0033328865529625956
- joint fr3_joint7: origin xyz=0.08771332066966753 -0.00012092092927270099 -0.00021330174425259079 rpy=1.571470088421461 0.0001348109342132342 0.0005679268841208079 -> xyz=0.08747489943452225 -0.0010959761553063266 0.00020303579109613634 rpy=1.5716067627690242 0.00011338979661758548 0.00040109418554127115

File: calibrated_urdf/fr3_2/step_2/model.urdf (robot description, URDF)
Before this commit: robot fr3, 15 links, 14 joints
Joints:
- joint ball_joint: origin xyz=0.0005804882467827815 0.00017580824461201 0.03223807954902509 rpy=0.0 0.0 0.0 -> xyz=0.000569829482925723 0.000178713331973003 0.03155177826612559 rpy=0.0 0.0 0.0
- joint fr3_finger_joint2: axis 0 -1 0 -> 0 1 0; origin xyz=0 0 0.0584 rpy=0 0 0 -> xyz=0 0 0.0584 rpy=0 0 3.141592653589793
- joint fr3_joint1: origin xyz=5.65828735332678e-18 2.6192086772817322e-17 0.333 rpy=6.735174465766389e-18 3.4048593312326387e-18 4.552229718360069e-17 -> xyz=2.0066905916350056e-16 -1.3675956436352349e-17 0.3330000000000001 rpy=8.939471544363453e-18 -6.541954763417535e-17 3.2696076431181047e-17
- joint fr3_joint2: origin xyz=-0.00027685062647461365 -7.650791676143057e-05 -1.1017630873410884e-17 rpy=-1.5690852800909436 0.008647594540282494 0.0002455741007457057 -> xyz=-0.00024560017837533274 -0.00018413846590304372 1.698372288445208e-17 rpy=-1.5688880810237205 0.008903221617202677 0.00036075831697496015
- joint fr3_joint3: origin xyz=0.0024679208933022154 -0.3159715454643631 5.7176998274987504e-05 rpy=1.568205472572578 -0.001116406452448498 0.006784581385823128 -> xyz=0.002500359991880905 -0.31588891922164175 3.244920587513935e-05 rpy=1.5681851754657918 -0.0010218307743303737 0.006787364459403446
- joint fr3_joint4: origin xyz=0.08236792578412418 -0.00034030907337044027 0.0006243726632184443 rpy=1.5675534812336325 0.0016743788782204029 0.0020092661447123268 -> xyz=0.08229574751680929 -0.0005195590560604383 0.0006987364875900003 rpy=1.5676264366903947 0.0016851209074791942 0.0020403664560433073
- joint fr3_joint5: origin xyz=-0.08204046581903031 0.3846305104765311 -0.0013208116023642321 rpy=-1.5713944717565103 0.0034011423798683636 -0.0011177311716949715 -> xyz=-0.08207811910450755 0.3846361326872398 -0.0015418615385886507 rpy=-1.571502414140622 0.0031056426044029184 -0.0009103574551739995
- joint fr3_joint6: origin xyz=0.0006405577078028358 0.0006213704515068757 0.0008939630970013438 rpy=1.5666140410821043 -0.00041142245320383166 0.0034491695847834233 -> xyz=0.000646734576377161 0.0009636158589815393 0.000924806021123695 rpy=1.56697844509155 -0.0008773013421369525 0.0035810247910971742
- joint fr3_joint7: origin xyz=0.08765444715507442 0.000343415694790559 -0.0001540329549196643 rpy=1.5712350885805113 8.556914472304246e-05 0.0003548984287086725 -> xyz=0.08755747889726417 -0.0003862654068421421 0.00011566679323867799 rpy=1.571346001046571 7.362689655808689e-05 0.00027299146342959254

File: calibrated_urdf/fr3_2/step_3/model.urdf (robot description, URDF)
Before this commit: robot fr3, 15 links, 14 joints
Joints:
- joint ball_joint: origin xyz=0.00058163176513666 0.00017110568660051997 0.032035093984850105 rpy=0.0 0.0 0.0 -> xyz=0.0005727299837121067 0.00017292333363062767 0.03164143469511594 rpy=0.0 0.0 0.0
- joint fr3_finger_joint2: axis 0 -1 0 -> 0 1 0; origin xyz=0 0 0.0584 rpy=0 0 0 -> xyz=0 0 0.0584 rpy=0 0 3.141592653589793
- joint fr3_joint1: origin xyz=3.710895219625396e-17 -8.602594479693649e-18 0.333 rpy=8.985903028001739e-18 -3.896253523572599e-17 -5.627116379310353e-17 -> xyz=3.210057584197411e-17 -1.3074045449295397e-17 0.3330000000000001 rpy=-8.121916481934434e-18 -6.637815225146384e-17 5.178385467344867e-17
- joint fr3_joint2: origin xyz=-0.000261450738052003 4.152260293607981e-06 -4.2313537066738635e-18 rpy=-1.5693812319217573 0.008309846293834383 9.371792218861651e-05 -> xyz=-0.00023669616307189241 -7.011674629893455e-05 1.766777250387578e-17 rpy=-1.5694982515547233 0.008434888133421727 0.00014793868502537287
- joint fr3_joint3: origin xyz=0.0024821393821360498 -0.3161460772079295 5.5167274581894415e-05 rpy=1.5682945293017505 -0.0015503409475926893 0.007112146198497874 -> xyz=0.0024812974849486792 -0.31608138959682336 1.8806441300969765e-05 rpy=1.5683542496870087 -0.001555168251681986 0.00710758214705765
- joint fr3_joint4: origin xyz=0.08234799280311385 0.00010146877357064115 0.0004063844389319755 rpy=1.5676069499426402 0.0015491372353014633 0.001883649468338221 -> xyz=0.0822257633023899 -4.63646366534432e-06 0.000423768129642051 rpy=1.5677096016093743 0.00146530321987359 0.0019669520733216553
- joint fr3_joint5: origin xyz=-0.08202558566962477 0.38467330278963474 -0.0007351564915896878 rpy=-1.5713800231690027 0.0035442960113612693 -0.0011826243625516764 -> xyz=-0.08204845684246093 0.3846702865950674 -0.0008402361743022892 rpy=-1.57144629766067 0.003397341424146344 -0.0010035343527974834
- joint fr3_joint6: origin xyz=0.000667936563000991 0.0004554430258604242 0.0007743675755292575 rpy=1.5662225970536015 -0.00014339616145485833 0.003562969033825572 -> xyz=0.0006841072828366817 0.0006262596632932238 0.0007890176922712335 rpy=1.566558851479323 -0.0003428234868287646 0.0035924610992054285
- joint fr3_joint7: origin xyz=0.08779762779622576 0.00020862438012274657 -0.00027384591017333274 rpy=1.5710115780035268 3.2583453597240656e-05 0.00012557865858040993 -> xyz=0.08776474644948352 -0.00019495727111732704 -0.00018106350854205598 rpy=1.5710715419888746 3.0035950257786534e-05 0.00010669271848338561

File: calibrated_urdf/fr3_2/step_4/model.urdf (robot description, URDF)
Before this commit: robot fr3, 15 links, 14 joints
Joints:
- joint ball_joint: origin xyz=0.000581779362790344 0.00017078378539145514 0.0318749511304747 rpy=0.0 0.0 0.0 -> xyz=0.0005730360200059966 0.00017248661896517427 0.031751185050378196 rpy=0.0 0.0 0.0
- joint fr3_finger_joint2: axis 0 -1 0 -> 0 1 0; origin xyz=0 0 0.0584 rpy=0 0 0 -> xyz=0 0 0.0584 rpy=0 0 3.141592653589793
- joint fr3_joint1: origin xyz=3.1777823966816564e-18 6.604463930052768e-18 0.333 rpy=5.844108460879476e-18 1.8062958579458646e-17 2.679816036714872e-17 -> xyz=-2.1551860152410533e-16 3.466379412284068e-18 0.3330000000000001 rpy=2.4720264225882587e-18 6.545184717647776e-17 1.0066016825856867e-17
- joint fr3_joint2: origin xyz=-0.00026107629855503687 2.7482713518423096e-05 -8.893042107392567e-18 rpy=-1.5694361059249653 0.00814109496606142 1.599465242612701e-05 -> xyz=-0.00023636675490102925 -3.171408963301376e-05 3.041231128627539e-17 rpy=-1.5696185407562486 0.008210958399695828 2.7813493976894585e-05
- joint fr3_joint3: origin xyz=0.00252407135557442 -0.31624308427600717 3.619197355645202e-05 rpy=1.5683173367389311 -0.0017183159062613281 0.007272996979078084 -> xyz=0.002528557020503575 -0.31620648766036147 -1.4984159053003679e-05 rpy=1.5684016448479587 -0.0017731455607090372 0.007309891705715417
- joint fr3_joint4: origin xyz=0.08234149717979959 0.0003513396069079546 0.0003028356098357084 rpy=1.5676184014834638 0.0014913386309645782 0.0017626899646134254 -> xyz=0.08220868988212866 0.0003194738824265976 0.00028586342227366306 rpy=1.5677326745390252 0.0013553051285632044 0.0018384954375648683
- joint fr3_joint5: origin xyz=-0.08201176450609714 0.3847123315326764 -0.000458977146233958 rpy=-1.5713585185051555 0.003563953918231571 -0.0012185398501815177 -> xyz=-0.08202406567204297 0.384714546232976 -0.0004781117970370225 rpy=-1.571402921365619 0.0034937738473749817 -0.0010652956253299802
- joint fr3_joint6: origin xyz=0.0006687091082321738 0.0003922719172020703 0.0007302600525192019 rpy=1.56619927154069 2.22220654686584e-06 0.0035677160149046494 -> xyz=0.0006847284750619545 0.00046201220443600126 0.000737471147760496 rpy=1.5665349784595053 -3.9408655076788224e-05 0.003531013141224253
- joint fr3_joint7: origin xyz=0.08786335402329959 6.29851364540537e-05 -0.0003565486498662301 rpy=1.570902974878879 5.559156908292331e-06 5.940811040122364e-06 -> xyz=0.08786441088940533 -5.723066621044474e-05 -0.0003738464873402999 rpy=1.570923374062213 5.647094083122981e-06 8.985060067905656e-06

File: calibrated_urdf/fr3_2/step_5/model.urdf (robot description, URDF)
Before this commit: robot fr3, 15 links, 14 joints
Joints:
- joint ball_joint: origin xyz=0.0005817897427710198 0.00017076431392279808 0.03181696256838364 rpy=0.0 0.0 0.0 -> xyz=0.0005730471232525534 0.00017246421521471098 0.03179576135750477 rpy=0.0 0.0 0.0
- joint fr3_finger_joint2: axis 0 -1 0 -> 0 1 0; origin xyz=0 0 0.0584 rpy=0 0 0 -> xyz=0 0 0.0584 rpy=0 0 3.141592653589793
- joint fr3_joint1: origin xyz=3.2503017915823636e-17 -1.0052584428671278e-17 0.333 rpy=9.835862032736894e-18 -1.568628146777241e-17 -9.300888715305458e-19 -> xyz=6.958869374967413e-17 3.7206810511837775e-18 0.333 rpy=2.0113251451119095e-18 -4.5173901919701175e-17 5.705740941573657e-17
- joint fr3_joint2: origin xyz=-0.0002610630417672176 3.162243216911802e-05 6.491857691235396e-18 rpy=-1.5694399183345502 0.008109347349404753 1.0266954813848713e-06 -> xyz=-0.0002363661414119994 -2.397097176040143e-05 3.2415594654458404e-18 rpy=-1.569627531576037 0.008165121152277102 1.992640972698194e-06
- joint fr3_joint3: origin xyz=0.002533495183565273 -0.31626197441515996 3.217901233781086e-05 rpy=1.5683189972748102 -0.0017477803894106437 0.00730424808627864 -> xyz=0.0025416874254174803 -0.3162341049030943 -2.277373293232744e-05 rpy=1.5684059469159568 -0.001813933435918177 0.007354648167490422
- joint fr3_joint4: origin xyz=0.08234090055495948 0.00040039919814801364 0.00028318793219997174 rpy=1.5676194275812498 0.001481487056437176 0.001736401255948335 -> xyz=0.08220731851774327 0.00039086001800762776 0.00025708364349779993 rpy=1.5677352085874752 0.0013346279635848702 0.0018045941861103785
- joint fr3_joint5: origin xyz=-0.08200856939548035 0.3847203771425275 -0.00040672740794162374 rpy=-1.5713567033269413 0.003565843461630894 -0.0012264927231521708 -> xyz=-0.08201778691104614 0.3847250851216539 -0.0004019899711809325 rpy=-1.5713980372610155 0.0035115086580737058 -0.0010810638186414354
- joint fr3_joint6: origin xyz=0.0006687445854766019 0.0003806617612789464 0.0007223020527509455 rpy=1.5661988055612805 3.25644008541223e-05 0.0035667292074115 -> xyz=0.0006845879920809151 0.0004274449250419267 0.0007274313178834408 rpy=1.5665350346686346 2.418741575571076e-05 0.0035147841764179544
- joint fr3_joint7: origin xyz=0.08787630243262287 7.798120106991974e-06 -0.0003730253641811346 rpy=1.5708821891077023 3.5812492014648904e-07 -1.7024685193937513e-05 -> xyz=0.08788500060358144 -7.255678665444132e-06 -0.0004160143465025743 rpy=1.5708917704419139 4.059015788202e-07 -1.2189018190717102e-05

File: urdf/fr3.urdf (robot description, URDF)
Before this commit: robot fr3, 15 links, 14 joints
Joints:
- joint ball_joint: origin xyz=0.000395598243266111 -7.962906613136055e-05 0.03180077705269587 rpy=0.0 0.0 0.0 -> xyz=7.773732033005863e-05 -4.214022515884392e-05 0.030128297908475325 rpy=0.0 0.0 0.0
- joint fr3_finger_joint2: axis 0 -1 0 -> 0 1 0; origin xyz=0 0 0.0584 rpy=0 0 0 -> xyz=0 0 0.0584 rpy=0 0 3.141592653589793
